File: Multi Edition/1.0A/SinESC-Multi-1.0A/SinESC-Multi-1.0A.kicad_pcb (KiCad board)
At the start: 4 copper layers, 30 x 15 mm, 84 parts, among them J1 Pad_3x2mm, J2 Pad_3x2mm, J3 Pad_3x2mm, J4 Pad_3x2mm, J5 Pad_3x2mm, J6 Pad_1.5mm_Square, Q1 BSC010N04LSI, Q2 BSC010N04LSI, Q3 BSC010N04LSI, Q4 BSC010N04LSI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

Commit message: PCB trace conditioning
Routing:
- net CUR_V: track 21.4 -> 20.5 mm
