File: Multi Edition/2.3B/SinESC-Multi-2.3B/SinESC-Multi-2.3B.sch (KiCad schematic (older format))
At the start: 84 parts, among them J1 Pad_3x2mm, J2 Pad_3x2mm, J3 Pad_3x2mm, J4 Pad_3x2mm, J5 Pad_3x2mm, J6 Pad_1.5mm_Square, Q1 BSC010N04LSI, Q2 BSC010N04LSI, Q3 BSC010N04LSI, Q4 BSC010N04LSI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

Commit message: Update R24 footprint & 3D model
Parts:
- R24: footprint Capacitor_SMD:C_0201_0603Metric -> Resistor_SMD:R_0201_0603Metric
Connections:
- net UART_RX_DSHOT renamed SINWIRE
Changed lines of the file:
@@
 NoConn ~ 1200 2900
 Text GLabel 1200 2800 0    50   Input ~ 0
-UART_RX_DSHOT
+SINWIRE
 Text GLabel 1200 2700 0    50   Output ~ 0
 UART_TX
@@
 	6150 4850 6350 4850
 Text GLabel 6350 5250 0    50   UnSpc ~ 0
-UART_RX_DSHOT
+SINWIRE
 $Comp
 L power:Earth #PWR022
@@
 F 0 "R24" V 9350 1150 50  0000 L CNN
 F 1 "52.3kΩ" V 9550 1150 50  0000 L CNN
-F 2 "Capacitor_SMD:C_0201_0603Metric" V 9490 1240 50  0001 C CNN
+F 2 "Resistor_SMD:R_0201_0603Metric" V 9490 1240 50  0001 C CNN
 F 3 "~" H 9450 1250 50  0001 C CNN
 F 4 "ERJ-1GNF5232C" H 9450 1250 50  0001 C CNN "Manufacturer Part #"

Commit message: Change resonator to part with interchangeable pins
Parts:
- Y1: Manufacturer Part # CSTNE8M00GH5C000R0 -> CSTNE8M00G550000R0
Changed lines of the file:
@@
 F 2 "Crystal:Resonator_SMD_muRata_CSTxExxV-3Pin_3.0x1.1mm" H 1000 1450 50  0001 C CNN
 F 3 "" H 1000 1450 50  0001 C CNN
-F 4 "CSTNE8M00GH5C000R0" H 1000 1450 50  0001 C CNN "Manufacturer Part #"
+F 4 "CSTNE8M00G550000R0" H 1000 1450 50  0001 C CNN "Manufacturer Part #"
 F 5 "-" H 1000 1450 50  0001 C CNN "Voltage Rating"
 	1    1000 1450
