File: Multi Edition/2.3B/SinESC-Multi-2.3B/SinESC-Multi-2.3B.kicad_pcb (KiCad board)
At the start: 4 copper layers, 30 x 15 mm, 84 parts, among them J1 Pad_3x2mm, J2 Pad_3x2mm, J3 Pad_3x2mm, J4 Pad_3x2mm, J5 Pad_3x2mm, J6 Pad_1.5mm_Square, Q1 BSC010N04LSI, Q2 BSC010N04LSI, Q3 BSC010N04LSI, Q4 BSC010N04LSI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

Commit message: Update R24 footprint & 3D model
Parts:
- R24: footprint Capacitor_SMD:C_0201_0603Metric -> Resistor_SMD:R_0201_0603Metric
Connections:
- net UART_RX_DSHOT renamed SINWIRE

Commit message: Update solder paste settings for improved yield (when assembled with stencil)
Parts:
- U4: value TMC6100-LA -> QFN37_7X7_TRI
