File: Multi Edition/SinESC-Multi/SinESC-Multi.kicad_pcb (KiCad board)
At the start: 4 copper layers, 30 x 15 mm, 84 parts, among them J1 Pad_3x2mm, J2 Pad_3x2mm, J3 Pad_3x2mm, J4 Pad_3x2mm, J5 Pad_3x2mm, J6 Pad_1.5mm_Square, Q1 BSC010N04LSI, Q2 BSC010N04LSI, Q3 BSC010N04LSI, Q4 BSC010N04LSI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

Commit message: Implement critical fix according to updated schematic, several other small updates (layout & silkscreen conditioning)
Parts:
- U4: value QFN37_7X7_TRI -> TMC6100-LA
- moved C29 0.30 mm to (37.6, 25.4)
- moved C28 0.25 mm to (39.1, 25.6)
Connections:
- C34 pad 2: Net-(C34-Pad2) -> +3V3
- C35 pad 2: Net-(C34-Pad2) -> +3V3
- L1 pad 2: Net-(C34-Pad2) -> +3V3
- R25 pad 2: Net-(C34-Pad2) -> +3V3
Routing:
- net +3V3: track 52.1 -> 68.2 mm
- net Net-(C34-Pad2): track 9.97 -> 0.00 mm
Other:
- board text added: "Designed by Erk S."
- board text added: "MULTI v2.3C"
- board text added: "Made in USA"
- board text removed: "Designed by SAR_mango Made in USA"
- board text removed: "MULTI v2.3B"
- board text removed: "Pre-Prod. S/N A0001"
