File: Multi Edition/SinESC-Multi/SinESC-Multi.kicad_pcb (KiCad board)
At the start: 4 copper layers, 30 x 15 mm, 84 parts, among them J1 Pad_3x2mm, J2 Pad_3x2mm, J3 Pad_3x2mm, J4 Pad_3x2mm, J5 Pad_3x2mm, J6 Pad_1.5mm_Square, Q1 BSC010N04LSI, Q2 BSC010N04LSI, Q3 BSC010N04LSI, Q4 BSC010N04LSI, Q5 BSC010N04LSI, Q6 BSC010N04LSI, U1 STM32F303CBT7, U2 MAX4239AUT, U3 MAX4239AUT, U4 TMC6100-LA, U5 MAX4239AUT, U6 TPS560430XDBVR, Y1 8MHz

Commit message: Update date reflected on sheet. Remove "Made in USA" from silkscreen to avoid customs issues when ordering boards from outside the U.S.
Other:
- board text removed: "Made in USA"

Commit message: Fix another issue in which the bootstrap capacitors were not connected to the source pins of the high-side FETs
Parts:
- renumbered C23 to C16, C24 to C17, C25 to C18, C16 to C19, C17 to C20, C18 to C21, C19 to C22, C20 to C23, C21 to C24, C22 to C25
Connections:
- C16 pad 1: Net-(C23-Pad1) -> U
- C17 pad 1: Net-(C24-Pad1) (its old number) -> V
- C18 pad 1: Net-(C25-Pad1) -> W
- U4 pad 32: Net-(C25-Pad1) -> W
- U4 pad 33: Net-(C24-Pad1) (its old number) -> V
- U4 pad 36: Net-(C23-Pad1) -> U
Routing:
- net U: track 13.4 -> 24.0 mm, vias 0 -> 2
- net W: track 18.9 -> 29.0 mm, vias 0 -> 2
- net V: track 23.8 -> 25.4 mm, vias 0 -> 1
- net Net-(C25-Pad1): track 1.29 -> 0.00 mm
- net Net-(C24-Pad1) (its old number): track 1.28 -> 0.00 mm
- net Net-(C23-Pad1): track 1.28 -> 0.00 mm
Other:
- board text added: "Designed in USA by Erk S."
- board text removed: "Designed by Erk S."
